Commit message: refresh for lab2

File: catkin_ws/src/me212_robot/model/me212_robot.xacro (robot description, xacro)
@@ -4,5 +4,5 @@
     <visual>
         <geometry>
-            <mesh filename="package://me212_robot/model/meshes/visual/me212_robot.stl"/>
+            <mesh scale="0.001 0.001 0.001" filename="package://me212_robot/model/meshes/visual/me212_robot.stl"/>
         </geometry>
         <material name="blue">
